Commit message: Changed laser to 270 degrees

File: src/unitree-go2-ros2/robots/descriptions/go2_description/xacro/laser.xacro (robot description, xacro)
@@ -1,4 +1,5 @@
 <?xml version="1.0"?>
 <robot xmlns:xacro="http://www.ros.org/wiki/xacro">
+    <!-- Visual laser link at original position -->
     <joint name="chassis_front_laser_joint" type="fixed">
         <axis xyz="0 0 1"/>
@@ -26,5 +27,19 @@
         </inertial>
     </link>
-    <gazebo reference="front_laser">
+    <!-- Sensor frame elevated by 0.3m for laser scanning -->
+    <joint name="front_laser_sensor_joint" type="fixed">
+        <axis xyz="0 0 1"/>
+        <origin rpy="0 0 0" xyz="0 0 0.3"/>
+        <parent link="front_laser"/>
+        <child link="front_laser_sensor"/>
+    </joint>
+    <link name="front_laser_sensor">
+        <inertial>
+        <mass value="1e-5"/>
+        <origin rpy="0 0 0" xyz="0 0 0"/>
+        <inertia ixx="1e-6" ixy="0" ixz="0" iyy="1e-6" iyz="0" izz="1e-6"/>
+        </inertial>
+    </link>
+    <gazebo reference="front_laser_sensor">
         <sensor name="front_laser_sensor" type="ray">
             <always_on>true</always_on>
@@ -37,6 +52,6 @@
                 <samples>240</samples>
                 <resolution>1.000000</resolution>
-                <min_angle>-1.570796</min_angle> // -90 degrees
-                <max_angle>1.570796</max_angle> // 90 degrees
+                <min_angle>-2.356194</min_angle> // -135 degrees. Total Field of View is 270 degrees
+                <max_angle>2.356194</max_angle>  // 135 degrees. Total Field of View is 270 degrees
                 </horizontal>
             </scan>
@@ -57,5 +72,5 @@
             </ros>
             <output_type>sensor_msgs/LaserScan</output_type>
-            <frame_name>front_laser</frame_name>
+            <frame_name>front_laser_sensor</frame_name>
             </plugin>
         </sensor>
